File: schematics/RobotLaberinto.kicad_sch (KiCad schematic)
At the start: 16 parts, among them J1 ALIM_EDU_CIAA, J2 ALIM_L298N

Commit message: updt pins on ide and sch
Connections:
- net GPIO5: now also R3.2, R4.1; no longer L298N_Shield1.10 (IN2)
- net GPIO8: now also L298N_Shield1.10 (IN2); no longer R3.2, R4.1
Other:
- note removed: "Diseño esquematico: Robot resuelve laberintos."
- moved on the sheet: CIAA-P1-1, CIAA-P2-1, HC-SR04-1, HC-SR04-2, HC-SR04-3, J1, J2, L298N_Shield1, MOT_A1, MOT_B1, R1, R2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
