File: schematics/robot2.kicad_sch (KiCad schematic)
At the start: 16 parts, among them J1 ALIM_EDU_CIAA, J2 ALIM_L298N

Commit message: update PCB
Connections:
- net GPIO5: now also L298N_Shield1.10 (IN2); no longer R3.2, R4.1
- net GPIO7: now also R3.2, R4.1; no longer HC-SR04-2.2 (Trigger)
- net GPIO8: now also HC-SR04-2.2 (Trigger); no longer L298N_Shield1.10 (IN2)
Changed lines of the file:
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@@
+		)
+	)
+	(global_label "GPIO5"
+		(shape input)
+		(at 186.69 107.95 180)
+		(fields_autoplaced yes)
+		(effects
+			(font
+				(size 1.27 1.27)
+			)
+			(justify right)
+		)
+		(property "Intersheetrefs" "${INTERSHEET_REFS}"
+			(at 178.02 107.95 0)
+			(effects
+				(font
+					(size 1.27 1.27)
+				)
+				(justify right)
+				(hide yes)
+			)
 		)
 	)
 	(global_label "GPIO8"
-		(shape input)
-		(at 186.69 107.95 180)
-		(fields_autoplaced yes)
-		(effects
-			(font
-				(size 1.27 1.27)
-			)
-			(justify right)
-		)
-		(property "Intersheetrefs" "${INTERSHEET_REFS}"
-			(at 178.02 107.95 0)
-			(effects
-				(font
-					(size 1.27 1.27)
-				)
-				(justify right)
-				(hide yes)
-			)
-		)
-	)
-	(global_label "GPIO7"
 		(shape input)
 		(at 99.06 54.61 180)
@@
 		)
 	)
-	(global_label "GPIO5"
+	(global_label "GPIO7"
 		(shape output)
 		(at 76.2 57.15 180)
