File: schematics/robot2.kicad_pcb (KiCad board)
At the start: 2 copper layers, 137 x 85.5 mm, 26 parts

Commit message: updt pcb
Parts:
- added ?: , , F.Cu at (104.5, 75.0)
- added ? (x2): , , F.Cu at (224.0, 81.5)
- added ?: , , F.Cu at (211.5, 81.5)
- added ?: , , F.Cu at (119.0, 75.0)
Routing:
- net GND: track 0.39 -> 27.4 mm

Commit message: updt pcb gnd
Parts:
- added ?: , , F.Cu at (138.5, 154.0)
- added ?: , , F.Cu at (126.0, 154.0)
- moved ? 59.5 mm to (141.5, 141.5)
- moved ? 59.5 mm to (168.6, 103.3) (x2)
- moved ? 59.5 mm to (156.1, 103.3)
- moved CIAA-P1-1 59.5 mm to (147.9, 119.8)
- moved CIAA-P2-1 59.5 mm to (76.3, 119.8)
- moved REF** 59.5 mm to (89.5, 135.5)
- moved ? 59.5 mm to (49.1, 96.8)
- moved ? 59.5 mm to (46.0, 162.3)
- moved ? 59.5 mm to (68.7, 153.3)
- moved ? 59.5 mm to (141.5, 144.0)
- moved ? 59.5 mm to (63.6, 96.8)
- moved HC-SR04-1 59.5 mm to (55.0, 120.3)
- moved HC-SR04-2 59.5 mm to (111.7, 162.0)
- moved HC-SR04-3 59.5 mm to (159.7, 120.3)
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Routing:
- net GND: track 27.4 -> 39.9 mm

Commit message: updt pcd
Parts:
- removed the ? at (168.6, 103.3)
Changed lines of the file:
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@@
 		(pad "1" thru_hole circle
 			(at 0 0 270)
-			(size 1.6 1.6)
+			(size 2.2 2.2)
 			(drill 0.7)
 			(layers "*.Cu" "*.Mask")
@@
 		(pad "2" thru_hole circle
 			(at 10.16 0 270)
-			(size 1.6 1.6)
+			(size 2.2 2.2)
 			(drill 0.7)
 			(layers "*.Cu" "*.Mask")
@@
 		(pad "1" thru_hole circle
 			(at -2.54 -2.54 270)
-			(size 2 2)
+			(size 2.2 2.2)
 			(drill 0.7)
 			(layers "*.Cu" "*.Mask")
@@
 		(pad "2" thru_hole circle
 			(at 0 -2.54 270)
-			(size 2 2)
+			(size 2.2 2.2)
 			(drill 0.7)
 			(layers "*.Cu" "*.Mask")
@@
 		(pad "3" thru_hole circle
 			(at 2.54 -2.54 270)
-			(size 2 2)
+			(size 2.2 2.2)
 			(drill 0.7)
 			(layers "*.Cu" "*.Mask")
@@
 		(pad "4" thru_hole circle
 			(at 5.08 -2.54 270)
-			(size 2 2)
+			(size 2.2 2.2)
 			(drill 0.7)
 			(layers "*.Cu" "*.Mask")
@@
 		(pad "1" thru_hole circle
 			(at 0 0 270)
-			(size 2 2)
+			(size 2.2 2.2)
 			(drill 0.7)
 			(layers "*.Cu" "*.Mask")
@@
 		(pad "1" thru_hole circle
 			(at 0 0 270)
-			(size 2 2)
+			(size 2.2 2.2)
 			(drill 0.7)
 			(layers "*.Cu" "*.Mask")
@@
 		(pad "2" thru_hole circle
 			(at 0 0 180)
-			(size 2 2)
+			(size 2.2 2.2)
 			(drill 0.7)
 			(layers "*.Cu" "*.Mask")
@@
 		(pad "1" thru_hole circle
 			(at 0 0 270)
-			(size 2 2)
+			(size 2.2 2.2)
 			(drill 0.7)
 			(layers "*.Cu" "*.Mask")
@@
 		(pad "2" thru_hole circle
 			(at 0 0 270)
-			(size 2 2)
+			(size 2.2 2.2)
 			(drill 0.7)
 			(layers "*.Cu" "*.Mask")
@@
 		(pad "1" thru_hole circle
 			(at 0 0)
-			(size 1.6 1.6)
+			(size 2.2 2.2)
 			(drill 0.7)
 			(layers "*.Cu" "*.Mask")
@@
 		(pad "2" thru_hole circle
 			(at 10.16 0)
-			(size 1.6 1.6)
+			(size 2.2 2.2)
 			(drill 0.7)
 			(layers "*.Cu" "*.Mask")
@@
 		(pad "1" thru_hole circle
 			(at -2.54 -2.54 270)
-			(size 2 2)
+			(size 2.2 2.2)
 			(drill 0.7)
 			(layers "*.Cu" "*.Mask")
@@
 		(pad "2" thru_hole circle
 			(at 0 -2.54 270)
-			(size 2 2)
+			(size 2.2 2.2)
 			(drill 0.7)
 			(layers "*.Cu" "*.Mask")
@@
 		(pad "3" thru_hole circle
 			(at 2.54 -2.54 270)
-			(size 2 2)
+			(size 2.2 2.2)
 			(drill 0.7)
 			(layers "*.Cu" "*.Mask")
@@
 		(pad "4" thru_hole circle
 			(at 5.08 -2.54 270)
-			(size 2 2)
+			(size 2.2 2.2)
 			(drill 0.7)
 			(layers "*.Cu" "*.Mask")
@@
 		(pad "1" thru_hole circle
 			(at 0 0 270)
-			(size 2 2)
+			(size 2.2 2.2)
 			(drill 0.7)
 			(layers "*.Cu" "*.Mask")
@@
 		(pad "1" thru_hole circle
 			(at 0 0 180)
-			(size 1.6 1.6)
+			(size 2.2 2.2)
 			(drill 0.7)
 			(layers "*.Cu" "*.Mask")
@@
 		(pad "2" thru_hole circle
 			(at 10.16 0 180)
-			(size 1.6 1.6)
+			(size 2.2 2.2)
 			(drill 0.7)
 			(layers "*.Cu" "*.Mask")
@@
 		(pad "1" thru_hole circle
 			(at 0 0)
-			(size 1.6 1.6)
+			(size 2.2 2.2)
 			(drill 0.7)
 			(layers "*.Cu" "*.Mask")
@@
 		(pad "2" thru_hole circle
 			(at 10.16 0)
-			(size 1.6 1.6)
+			(size 2.2 2.2)
 			(drill 0.7)
 			(layers "*.Cu" "*.Mask")
@@
 		(pad "1" thru_hole circle
 			(at 0 0 180)
-			(size 1.6 1.6)
+			(size 2.2 2.2)
 			(drill 0.7)
 			(layers "*.Cu" "*.Mask")
@@
 		(pad "2" thru_hole circle
 			(at 10.16 0 180)
-			(size 1.6 1.6)
+			(size 2.2 2.2)
 			(drill 0.7)
 			(layers "*.Cu" "*.Mask")
@@
 		(pad "1" thru_hole circle
 			(at -2.54 -2.54)
-			(size 2 2)
+			(size 2.2 2.2)
 			(drill 0.7)
 			(layers "*.Cu" "*.Mask")
@@
 		(pad "2" thru_hole circle
 			(at 0 -2.54)
-			(size 2 2)
+			(size 2.2 2.2)
 			(drill 0.7)
 			(layers "*.Cu" "*.Mask")
@@
 		(pad "3" thru_hole circle
 			(at 2.54 -2.54)
-			(size 2 2)
+			(size 2.2 2.2)
 			(drill 0.7)
 			(layers "*.Cu" "*.Mask")
@@
 		(pad "4" thru_hole circle
 			(at 5.08 -2.54)
-			(size 2 2)
+			(size 2.2 2.2)
 			(drill 0.7)
 			(layers "*.Cu" "*.Mask")
@@
 		(pad "1" thru_hole circle
 			(at 0 0 180)
-			(size 1.6 1.6)
+			(size 2.2 2.2)
 			(drill 0.7)
 			(layers "*.Cu" "*.Mask")
@@
 		(pad "2" thru_hole circle
 			(at 10.16 0 180)
-			(size 1.6 1.6)
+			(size 2.2 2.2)
 			(drill 0.7)
 			(layers "*.Cu" "*.Mask")
@@
 		(pad "1" thru_hole circle
 			(at 0 0 180)
-			(size 2 2)
+			(size 2.2 2.2)
 			(drill 0.7)
 			(layers "*.Cu" "*.Mask")
 			(remove_unused_layers no)
 			(net 78 "GPIO6")
-			(pinfunction "Vcc")
-			(pintype "power_in")
-		)
-		(embedded_fonts no)
-	)
-	(footprint ""
-		(layer "F.Cu")
-		(at 168.602 103.29)
-		(property "Reference" ""
-			(at 0 0 0)
-			(layer "F.SilkS")
-			(effects
-				(font
-					(size 1.27 1.27)
-					(thickness 0.15)
-				)
-			)
-		)
-		(property "Value" ""
-			(at 0 0 0)
-			(layer "F.Fab")
-			(effects
-				(font
-					(size 1.27 1.27)
-					(thickness 0.15)
-				)
-			)
-		)
-		(property "Datasheet" ""
-			(at 0 0 0)
-			(layer "F.Fab")
-			(hide yes)
-			(effects
-				(font
-					(size 1.27 1.27)
-					(thickness 0.15)
-				)
-			)
-		)
-		(property "Description" ""
-			(at 0 0 0)
-			(layer "F.Fab")
-			(hide yes)
-			(effects
-				(font
-					(size 1.27 1.27)
-					(thickness 0.15)
-				)
-			)
-		)
-		(pad "1" thru_hole circle
-			(at 0 0 270)
-			(size 2 2)
-			(drill 0.7)
-			(layers "*.Cu" "*.Mask")
-			(remove_unused_layers no)
-			(net 1 "GND")
 			(pinfunction "Vcc")
 			(pintype "power_in")
@@
 		(pad "2" thru_hole circle
 			(at 0 0 270)
-			(size 2 2)
-			(drill 0.7)
-			(layers "*.Cu" "*.Mask")
+			(size 2.2 2.2)
+			(drill 0.7)
+			(layers "*.Cu" "*.Mask")
